File: hardware/NEO-6M-0-001-tryout.kicad_pcb (KiCad board)
At the start: 2 copper layers, 24 parts, among them J1 IPEX, J2 BAT_CONN, U1 24AA32A, U2 TTL_TERMINAL, U3 UBLOX-NEO-6M-0-001, U4 AMS1117-3.3, U5 USB_Micro

Commit message: update,
Parts:
- moved R3 2.33 mm to (49.7, 44.6), turned to 270 degrees
- moved J1 0.89 mm to (41.8, 45.8)
- moved L1 0.71 mm to (46.3, 45.7), turned to 0 degrees
Routing:
- net GND: track 0.00 -> 148.3 mm
- net +3V3: track 0.00 -> 70.7 mm
- net +5V: track 0.00 -> 21.8 mm
- net Net-(C2-Pad1): track 0.00 -> 20.9 mm
- net Net-(J2-Pad1): track 0.00 -> 14.0 mm
- net /TX: track 0.00 -> 11.2 mm
- net Net-(J1-Pad1): track 0.00 -> 11.0 mm
- net /RX: track 0.00 -> 9.62 mm
- net /GSCL: track 0.00 -> 8.97 mm
- net /GSDA: track 0.00 -> 8.54 mm
- net Net-(R3-Pad1): track 0.00 -> 7.35 mm
- net Net-(C1-Pad1): track 0.00 -> 5.08 mm, vias 0 -> 1
- net Net-(R1-Pad2): track 0.00 -> 3.34 mm, vias 0 -> 1
- net Net-(D2-Pad1): track 0.00 -> 2.81 mm, vias 0 -> 1
- net Net-(D3-Pad1): track 0.00 -> 2.25 mm, vias 0 -> 1
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